File: Hardware/Power-Control.sch (KiCad schematic (older format))
At the start: 20 parts, among them K1 SANYOU_SRD_Form_A, Q1 AO3400A, U2 MOC3023M, U3 MOC3023M, U4 H11AA1

Commit message: Funktionalität für Verbraucher hinzugefügt. PID-Controller hinzugefügt. MAX31855 Driver hinzugefügt. Minimalbeispiel für Reflow-Prozess erstellt.
Parts:
- R10, R9: LCSC C25117 -> C23179
Changed lines of the file:
@@
 F 2 "Resistor_SMD:R_0603_1608Metric" H 5000 1800 50  0001 C CNN
 F 3 "~" H 5000 1800 50  0001 C CNN
-F 4 "C25117" H 5000 1800 50  0001 C CNN "LCSC"
+F 4 "C23179" H 5000 1800 50  0001 C CNN "LCSC"
 	1    5000 1800
 	0    1    1    0
@@
 F 2 "Resistor_SMD:R_0603_1608Metric" H 5000 3750 50  0001 C CNN
 F 3 "~" H 5000 3750 50  0001 C CNN
-F 4 "C25117" H 5000 3750 50  0001 C CNN "LCSC"
+F 4 "C23179" H 5000 3750 50  0001 C CNN "LCSC"
 	1    5000 3750
 	0    1    1    0
